File: PCB/MainBoardV2/Power.sch (KiCad schematic (older format))
At the start: 51 parts, among them Q17 DMP3099L-7, Q18 NTR4003NT3G, Q2 DMP3099L-7, Q3 NTR4003NT3G, Q4 DMP3099L-7, SW2 SWITCH_DPDT, SW4 SWITCH_DPDT, U1 LTC2992, U2 AZ2117H, U3 AZ2117H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

Commit message: Layout Done - Needs TPs Still
Parts:
- R9: value 10 -> 10m
Changed lines of the file:
@@
 $EndComp
 $Comp
-L GND #PWR25
+L GND #PWR026
 U 1 1 5A389D93
 P 1400 2500
-F 0 "#PWR25" H 1400 2250 50  0001 C CNN
+F 0 "#PWR026" H 1400 2250 50  0001 C CNN
 F 1 "GND" H 1500 2400 50  0000 C CNN
 F 2 "" H 1400 2500 50  0000 C CNN
@@
 $EndComp
 $Comp
-L GND #PWR26
+L GND #PWR027
 U 1 1 5A389DCA
 P 1400 3150
-F 0 "#PWR26" H 1400 2900 50  0001 C CNN
+F 0 "#PWR027" H 1400 2900 50  0001 C CNN
 F 1 "GND" H 1500 3050 50  0000 C CNN
 F 2 "" H 1400 3150 50  0000 C CNN
@@
 $EndComp
 $Comp
-L GND #PWR28
+L GND #PWR028
 U 1 1 5A38AD41
 P 2350 3600
-F 0 "#PWR28" H 2350 3350 50  0001 C CNN
+F 0 "#PWR028" H 2350 3350 50  0001 C CNN
 F 1 "GND" H 2350 3450 50  0000 C CNN
 F 2 "" H 2350 3600 50  0000 C CNN
@@
 $EndComp
 $Comp
-L GND #PWR33
+L GND #PWR029
 U 1 1 5A38F8D3
 P 4600 2500
-F 0 "#PWR33" H 4600 2250 50  0001 C CNN
+F 0 "#PWR029" H 4600 2250 50  0001 C CNN
 F 1 "GND" H 4600 2350 50  0000 C CNN
 F 2 "" H 4600 2500 50  0000 C CNN
@@
 $EndComp
 $Comp
-L GND #PWR29
+L GND #PWR030
 U 1 1 5A390EFC
 P 2700 3750
-F 0 "#PWR29" H 2700 3500 50  0001 C CNN
+F 0 "#PWR030" H 2700 3500 50  0001 C CNN
 F 1 "GND" H 2700 3600 50  0000 C CNN
 F 2 "" H 2700 3750 50  0000 C CNN
@@
 $EndComp
 $Comp
-L GND #PWR30
+L GND #PWR031
 U 1 1 5A3921C3
 P 3250 3150
-F 0 "#PWR30" H 3250 2900 50  0001 C CNN
+F 0 "#PWR031" H 3250 2900 50  0001 C CNN
 F 1 "GND" H 3250 3000 50  0000 C CNN
 F 2 "" H 3250 3150 50  0000 C CNN
@@
 $EndComp
 $Comp
-L GND #PWR42
+L GND #PWR032
 U 1 1 5A3978FC
 P 8600 3200
-F 0 "#PWR42" H 8600 2950 50  0001 C CNN
+F 0 "#PWR032" H 8600 2950 50  0001 C CNN
 F 1 "GND" H 8600 3050 50  0000 C CNN
 F 2 "" H 8600 3200 50  0000 C CNN
@@
 $EndComp
 $Comp
-L GND #PWR43
+L GND #PWR033
 U 1 1 5A397C6D
 P 8600 4350
-F 0 "#PWR43" H 8600 4100 50  0001 C CNN
+F 0 "#PWR033" H 8600 4100 50  0001 C CNN
 F 1 "GND" H 8600 4200 50  0000 C CNN
 F 2 "" H 8600 4350 50  0000 C CNN
@@
 $EndComp
 $Comp
-L GND #PWR41
+L GND #PWR034
 U 1 1 5A398674
 P 8150 4750
-F 0 "#PWR41" H 8150 4500 50  0001 C CNN
+F 0 "#PWR034" H 8150 4500 50  0001 C CNN
 F 1 "GND" H 8150 4600 50  0000 C CNN
 F 2 "" H 8150 4750 50  0000 C CNN
@@
 $EndComp
 $Comp
-L GND #PWR40
+L GND #PWR035
 U 1 1 5A3991C6
 P 8150 3650
-F 0 "#PWR40" H 8150 3400 50  0001 C CNN
+F 0 "#PWR035" H 8150 3400 50  0001 C CNN
 F 1 "GND" H 8150 3500 50  0000 C CNN
 F 2 "" H 8150 3650 50  0000 C CNN
@@
 $EndComp
 $Comp
-L GND #PWR36
+L GND #PWR036
 U 1 1 5A3A5706
 P 6850 3200
-F 0 "#PWR36" H 6850 2950 50  0001 C CNN
+F 0 "#PWR036" H 6850 2950 50  0001 C CNN
 F 1 "GND" H 6850 3050 50  0000 C CNN
 F 2 "" H 6850 3200 50  0000 C CNN
@@
 $EndComp
 $Comp
-L GND #PWR37
+L GND #PWR037
 U 1 1 5A3A67D1
 P 6850 4350
-F 0 "#PWR37" H 6850 4100 50  0001 C CNN
+F 0 "#PWR037" H 6850 4100 50  0001 C CNN
 F 1 "GND" H 6850 4200 50  0000 C CNN
 F 2 "" H 6850 4350 50  0000 C CNN
@@
 $EndComp
 $Comp
-L GND #PWR38
+L GND #PWR038
 U 1 1 5A38AA5C
 P 7000 1900
-F 0 "#PWR38" H 7000 1650 50  0001 C CNN
+F 0 "#PWR038" H 7000 1650 50  0001 C CNN
 F 1 "GND" H 7000 1750 50  0000 C CNN
 F 2 "" H 7000 1900 50  0000 C CNN
@@
 P 6750 1600
 F 0 "R9" V 6830 1600 50  0000 C CNN
-F 1 "10" V 6750 1600 50  0000 C CNN
+F 1 "10m" V 6750 1600 50  0000 C CNN
 F 2 "Resistors_SMD:R_0805_HandSoldering" V 6680 1600 50  0001 C CNN
 F 3 "" H 6750 1600 50  0000 C CNN
@@
 $EndComp
 $Comp
-L GND #PWR44
+L GND #PWR039
 U 1 1 5A38B18F
 P 8750 2400
-F 0 "#PWR44" H 8750 2150 50  0001 C CNN
+F 0 "#PWR039" H 8750 2150 50  0001 C CNN
 F 1 "GND" H 8750 2250 50  0000 C CNN
 F 2 "" H 8750 2400 50  0000 C CNN
@@
 $EndComp
 $Comp
-L GND #PWR39
+L GND #PWR040
 U 1 1 5A38B2C3
 P 7650 2400
-F 0 "#PWR39" H 7650 2150 50  0001 C CNN
+F 0 "#PWR040" H 7650 2150 50  0001 C CNN
 F 1 "GND" H 7650 2250 50  0000 C CNN
 F 2 "" H 7650 2400 50  0000 C CNN
@@
 Switch_FB
 $Comp
-L GND #PWR45
+L GND #PWR041
 U 1 1 5A38F87B
 P 9750 2600
-F 0 "#PWR45" H 9750 2350 50  0001 C CNN
+F 0 "#PWR041" H 9750 2350 50  0001 C CNN
 F 1 "GND" H 9750 2450 50  0000 C CNN
 F 2 "" H 9750 2600 50  0000 C CNN
@@
 +6.5V
 $Comp
-L GND #PWR46
+L GND #PWR042
 U 1 1 5A39294C
 P 10300 2250
-F 0 "#PWR46" H 10300 2000 50  0001 C CNN
+F 0 "#PWR042" H 10300 2000 50  0001 C CNN
 F 1 "GND" H 10300 2100 50  0000 C CNN
 F 2 "" H 10300 2250 50  0000 C CNN
@@
 $EndComp
 $Comp
-L GND #PWR32
+L GND #PWR043
 U 1 1 5A6F3B2D
 P 4200 7300
-F 0 "#PWR32" H 4200 7050 50  0001 C CNN
+F 0 "#PWR043" H 4200 7050 50  0001 C CNN
 F 1 "GND" H 4200 7150 50  0000 C CNN
 F 2 "" H 4200 7300 50  0000 C CNN
@@
 $EndComp
 $Comp
-L GND #PWR35
+L GND #PWR044
 U 1 1 5A6F48B4
 P 5950 7300
-F 0 "#PWR35" H 5950 7050 50  0001 C CNN
+F 0 "#PWR044" H 5950 7050 50  0001 C CNN
 F 1 "GND" H 5950 7150 50  0000 C CNN
 F 2 "" H 5950 7300 50  0000 C CNN
@@
 $EndComp
 $Comp
-L GND #PWR34
+L GND #PWR045
 U 1 1 5A736B75
 P 4950 3700
-F 0 "#PWR34" H 4950 3450 50  0001 C CNN
+F 0 "#PWR045" H 4950 3450 50  0001 C CNN
 F 1 "GND" H 4950 3550 50  0000 C CNN
 F 2 "" H 4950 3700 50  0000 C CNN
@@
 $EndComp
 $Comp
-L GND #PWR31
+L GND #PWR046
 U 1 1 5A768705
 P 3500 4700
-F 0 "#PWR31" H 3500 4450 50  0001 C CNN
+F 0 "#PWR046" H 3500 4450 50  0001 C CNN
 F 1 "GND" H 3600 4600 50  0000 C CNN
 F 2 "" H 3500 4700 50  0000 C CNN
@@
 $EndComp
 $Comp
-L GND #PWR27
+L GND #PWR047
 U 1 1 5A76A3C6
 P 1900 4750
-F 0 "#PWR27" H 1900 4500 50  0001 C CNN
+F 0 "#PWR047" H 1900 4500 50  0001 C CNN
 F 1 "GND" H 1900 4600 50  0000 C CNN
 F 2 "" H 1900 4750 50  0000 C CNN
