File: PCB/MainBoardV2/MSP430.sch (KiCad schematic (older format))
At the start: 30 parts, among them Q12 NTR4003NT3G, Q14 NTR4003NT3G, Q15 NTR4003NT3G, SW1 PTS645SM43SMTR92 LFS, U8 MSP430FR5994, U9 ASEMB-24MHZ-XY-T, Y1 32.768 kHz

Commit message: Board Completed. Needs Review
Connections:
- net RESET_VIDEO_PI: no longer names the net of U8.67 (P5.6_UCA2CLK_TA4.0_SMCLK)
- no-connect marks 33 -> 34
Changed lines of the file:
@@
 $EndComp
 $Comp
-L GND #PWR080
+L GND #PWR079
 U 1 1 5A00F83B
 P 1300 1400
-F 0 "#PWR080" H 1300 1150 50  0001 C CNN
+F 0 "#PWR079" H 1300 1150 50  0001 C CNN
 F 1 "GND" H 1300 1250 50  0000 C CNN
 F 2 "" H 1300 1400 50  0000 C CNN
@@
 $EndComp
 $Comp
-L GND #PWR081
+L GND #PWR080
 U 1 1 5A00F879
 P 9450 1800
-F 0 "#PWR081" H 9450 1550 50  0001 C CNN
+F 0 "#PWR080" H 9450 1550 50  0001 C CNN
 F 1 "GND" H 9450 1650 50  0000 C CNN
 F 2 "" H 9450 1800 50  0000 C CNN
@@
 RST_SBWTDIO_HOST
 $Comp
-L GND #PWR082
+L GND #PWR081
 U 1 1 5A00F8A8
 P 7050 6250
-F 0 "#PWR082" H 7050 6000 50  0001 C CNN
+F 0 "#PWR081" H 7050 6000 50  0001 C CNN
 F 1 "GND" H 7050 6100 50  0000 C CNN
 F 2 "" H 7050 6250 50  0000 C CNN
@@
 $EndComp
 $Comp
-L GND #PWR083
+L GND #PWR082
 U 1 1 5A00F8FE
 P 5700 7450
-F 0 "#PWR083" H 5700 7200 50  0001 C CNN
+F 0 "#PWR082" H 5700 7200 50  0001 C CNN
 F 1 "GND" H 5700 7300 50  0000 C CNN
 F 2 "" H 5700 7450 50  0000 C CNN
@@
 $EndComp
 $Comp
-L GND #PWR084
+L GND #PWR083
 U 1 1 5A00F91F
 P 10000 3350
-F 0 "#PWR084" H 10000 3100 50  0001 C CNN
+F 0 "#PWR083" H 10000 3100 50  0001 C CNN
 F 1 "GND" H 10000 3200 50  0000 C CNN
 F 2 "" H 10000 3350 50  0000 C CNN
@@
 NoConn ~ 8800 2750
 $Comp
-L GND #PWR085
+L GND #PWR084
 U 1 1 5A00F92C
 P 8700 3050
-F 0 "#PWR085" H 8700 2800 50  0001 C CNN
+F 0 "#PWR084" H 8700 2800 50  0001 C CNN
 F 1 "GND" H 8700 2900 50  0000 C CNN
 F 2 "" H 8700 3050 50  0000 C CNN
@@
 $EndComp
 $Comp
-L GND #PWR086
+L GND #PWR085
 U 1 1 5A376B4C
 P 3100 7200
-F 0 "#PWR086" H 3100 6950 50  0001 C CNN
+F 0 "#PWR085" H 3100 6950 50  0001 C CNN
 F 1 "GND" H 3100 7050 50  0000 C CNN
 F 2 "" H 3100 7200 50  0000 C CNN
@@
 $EndComp
 $Comp
-L GND #PWR087
+L GND #PWR086
 U 1 1 5A376B5B
 P 3550 7450
-F 0 "#PWR087" H 3550 7200 50  0001 C CNN
+F 0 "#PWR086" H 3550 7200 50  0001 C CNN
 F 1 "GND" H 3700 7400 50  0000 C CNN
 F 2 "" H 3550 7450 50  0000 C CNN
@@
 Wire Wire Line
 	3550 7000 3550 7150
-Text GLabel 2050 4300 0    39   Input ~ 0
-RESET_VIDEO_PI
 Wire Wire Line
 	9100 1800 9800 1800
@@
 	10500 4400 10400 4400
 Connection ~ 10000 4400
+NoConn ~ 2050 4300
 $EndSCHEMATC

Commit message: Added BOM, Couple Fixes, Couple Misc Documents
Parts:
- C23, C27, C28, C29: value 100nF -> 0.1uF
- C24: value 1000pF -> 1nF
- R55: value 80 -> 100
- renumbered U9 to Y2
Connections:
- net +3.3V: now also R46.1
- net +5V: no longer R46.1
- net MULTIPLEX_A0: no longer names the net of U8.17 (P1.4_TB0.1_UCA0STE_A4_C4)
- net MULTIPLEX_A1 renamed MSP_GPIO_CB
- no-connect marks 34 -> 35
Changed lines of the file:
@@
 P 1300 1250
 F 0 "C23" H 1325 1350 50  0000 L CNN
-F 1 "100nF" H 1325 1150 50  0000 L CNN
+F 1 "0.1uF" H 1325 1150 50  0000 L CNN
 F 2 "Capacitors_SMD:C_0805_HandSoldering" H 1338 1100 50  0001 C CNN
 F 3 "" H 1300 1250 50  0000 C CNN
@@
 Text GLabel 2050 2200 0    39   Input ~ 0
 DAQCS_CS
-Text GLabel 2050 2300 0    39   Input ~ 0
-MULTIPLEX_A0
 Text GLabel 2050 2400 0    39   Input ~ 0
-MULTIPLEX_A1
+MSP_GPIO_CB
 Text GLabel 2050 2500 0    39   Input ~ 0
 DAQCS_MOSI
@@
 P 5700 7200
 F 0 "C27" H 5725 7300 50  0000 L CNN
-F 1 "100nF" H 5725 7100 50  0000 L CNN
+F 1 "0.1uF" H 5725 7100 50  0000 L CNN
 F 2 "Capacitors_SMD:C_0805_HandSoldering" H 5738 7050 50  0001 C CNN
 F 3 "" H 5700 7200 50  0000 C CNN
@@
 P 6100 7200
 F 0 "C28" H 6125 7300 50  0000 L CNN
-F 1 "100nF" H 6125 7100 50  0000 L CNN
+F 1 "0.1uF" H 6125 7100 50  0000 L CNN
 F 2 "Capacitors_SMD:C_0805_HandSoldering" H 6138 7050 50  0001 C CNN
 F 3 "" H 6100 7200 50  0000 C CNN
@@
 P 6500 7200
 F 0 "C29" H 6525 7300 50  0000 L CNN
-F 1 "100nF" H 6525 7100 50  0000 L CNN
+F 1 "0.1uF" H 6525 7100 50  0000 L CNN
 F 2 "Capacitors_SMD:C_0805_HandSoldering" H 6538 7050 50  0001 C CNN
 F 3 "" H 6500 7200 50  0000 C CNN
@@
 High-Freq. Oscillator
 $Comp
-L ASEMB-24MHZ-XY-T U9
+L ASEMB-24MHZ-XY-T Y2
 U 1 1 5A00F90A
 P 9350 2850
-F 0 "U9" H 9350 3100 60  0000 C CNN
+F 0 "Y2" H 9350 3100 60  0000 C CNN
 F 1 "ASEMB-24MHZ-XY-T" H 9400 2600 60  0000 C CNN
 F 2 "Dans_Parts:ASEMB-24MHZ" H 9350 2850 60  0001 C CNN
@@
 P 3550 7300
 F 0 "C24" H 3575 7400 50  0000 L CNN
-F 1 "1000pF" H 3200 7400 50  0000 L CNN
+F 1 "1nF" H 3350 7400 50  0000 L CNN
 F 2 "Capacitors_SMD:C_0805_HandSoldering" H 3588 7150 50  0001 C CNN
 F 3 "" H 3550 7300 50  0000 C CNN
@@
 P 9650 5250
 F 0 "R55" V 9550 5250 50  0000 C CNN
-F 1 "80" V 9650 5250 50  0000 C CNN
+F 1 "100" V 9650 5250 50  0000 C CNN
 F 2 "Resistors_SMD:R_0805_HandSoldering" V 9580 5250 50  0001 C CNN
 F 3 "" H 9650 5250 50  0000 C CNN
@@
 $EndComp
 Text GLabel 10500 4400 2    39   Input ~ 0
-+5V
++3.3V
 Wire Wire Line
 	10500 4400 10400 4400
 Connection ~ 10000 4400
 NoConn ~ 2050 4300
+NoConn ~ 2050 2300
 $EndSCHEMATC
