File: PCB/MainBoardV2/Sensors.sch (KiCad schematic (older format))
At the start: 8 parts, among them U6 LSM9DS1, U7 BME280

Commit message: Added BOM, Couple Fixes, Couple Misc Documents
Parts:
- C18: value 10uF -> 0.1uF
- C20: value 100nF -> 0.1uF
Changed lines of the file:
@@
 P 2250 1550
 F 0 "C18" H 2000 1600 50  0000 L CNN
-F 1 "10uF" H 1950 1450 50  0000 L CNN
+F 1 "0.1uF" H 1950 1450 50  0000 L CNN
 F 2 "Capacitors_SMD:C_0805_HandSoldering" H 2288 1400 50  0001 C CNN
 F 3 "" H 2250 1550 50  0000 C CNN
@@
 P 2400 2200
 F 0 "C20" H 2425 2300 50  0000 L CNN
-F 1 "100nF" H 2425 2100 50  0000 L CNN
+F 1 "0.1uF" H 2425 2100 50  0000 L CNN
 F 2 "Capacitors_SMD:C_0805_HandSoldering" H 2438 2050 50  0001 C CNN
 F 3 "" H 2400 2200 50  0000 C CNN
