File: PCB/MainBoardV2/mainBoardV2.kicad_pcb (KiCad board)
At the start: 2 copper layers, 102 x 108 mm, 175 parts, among them J1 Pi0_1, J10 Backup_Battery, J11 External_Temp, J12 Comms_I2C, J13 Main_Monitoring, J14 2S_Primary_Batt, J15 2S_Backup_Batt, J16 Programming, J17 To_Balloon, J18 Motor_Batt_Monitoring, J19 PI 3 RESET, J2 Pi0_2, J20 RESET_VIDEO_PI, J3 Pi0_3, J4 To_Motor, J5 To_Center_Board, J6 Pi0_4, J7 From_Motor, J8 Main_Battery, J9 Comms_SPI, Q1 NTD20N03L27T4G, Q12 NTR4003NT3G, Q14 NTR4003NT3G, Q15 NTR4003NT3G, Q17 DMP3099L-7, Q18 NTR4003NT3G, Q2 DMP3099L-7, Q3 NTR4003NT3G, Q4 DMP3099L-7, Q5 NTR4003NT3G, Q6 NTR4003NT3G, Q7 NTR4003NT3G, Q8 NTR4003NT3G, Q9 NTR4003NT3G, SW1 PTS645SM43SMTR92 LFS, SW2 SWITCH_DPDT, SW3 PTS645SM43SMTR92 LFS, SW4 SWITCH_DPDT, U1 LTC2992, U10 AOZ8318DI, U11 AOZ8318DI, U12 AOZ8318DI, U2 AZ2117H, U3 AZ2117H, U4 LT8609, U5 Teensy3.6, U6 LSM9DS1, U7 BME280, U8 MSP430FR5994, U9 ASEMB-24MHZ-XY-T, Y1 32.768 kHz

Commit message: Layout Done - Needs TPs Still
Parts:
- removed D18: SBRT5A50SA-13, Dans_Parts:DO-214AC_Schottky
- added D11: SBRT5A50SA-13, Dans_Parts:DO-214AC_Schottky, F.Cu at (97.1, 71.9)
- added J21: Ethernet_Switch_PWR, Dans_Parts:2-Pin_Molex_Horizontal, F.Cu at (74.3, 25.3)
- added REF**: Via-0.6mm, Dans_Parts:Via-0.6mm, F.Cu at (79.9, 68.0)
- added REF**: Via-0.6mm, Dans_Parts:Via-0.6mm, F.Cu at (94.5, 79.6)
- added REF**: Via-0.6mm, Dans_Parts:Via-0.6mm, F.Cu at (98.1, 121.4)
- added REF**: Via-0.6mm, Dans_Parts:Via-0.6mm, F.Cu at (108.5, 120.0)
- added REF**: Via-0.6mm, Dans_Parts:Via-0.6mm, F.Cu at (69.8, 73.1)
- added REF**: Via-0.6mm, Dans_Parts:Via-0.6mm, F.Cu at (64.0, 75.9)
- added REF**: Via-0.6mm, Dans_Parts:Via-0.6mm, F.Cu at (72.5, 71.0)
- added REF**: Via-0.6mm, Dans_Parts:Via-0.6mm, F.Cu at (67.7, 73.1)
- added REF**: Via-0.6mm, Dans_Parts:Via-0.6mm, F.Cu at (57.0, 75.8)
- added REF**: Via-0.6mm, Dans_Parts:Via-0.6mm, F.Cu at (61.5, 75.9)
- added REF**: Via-0.6mm, Dans_Parts:Via-0.6mm, F.Cu at (57.1, 122.9)
- added REF**: Via-0.6mm, Dans_Parts:Via-0.6mm, F.Cu at (105.0, 125.6)
- added REF**: Via-0.6mm, Dans_Parts:Via-0.6mm, F.Cu at (89.8, 79.7)
- added REF**: Via-0.6mm, Dans_Parts:Via-0.6mm, F.Cu at (23.3, 102.0)
- added REF**: Via-0.6mm, Dans_Parts:Via-0.6mm, F.Cu at (45.1, 102.3)
- added REF**: Via-0.6mm, Dans_Parts:Via-0.6mm, F.Cu at (58.9, 64.1)
- added REF**: Via-0.6mm, Dans_Parts:Via-0.6mm, F.Cu at (71.0, 63.8)
- added REF**: Via-0.6mm, Dans_Parts:Via-0.6mm, F.Cu at (64.0, 81.1)
- added REF**: Via-0.6mm, Dans_Parts:Via-0.6mm, F.Cu at (71.8, 64.8)
- added REF**: Via-0.6mm, Dans_Parts:Via-0.6mm, F.Cu at (57.1, 67.1)
- added REF**: Via-0.6mm, Dans_Parts:Via-0.6mm, F.Cu at (56.9, 71.6)
- added REF**: Via-0.6mm, Dans_Parts:Via-0.6mm, F.Cu at (49.3, 125.6)
- added REF**: Via-0.6mm, Dans_Parts:Via-0.6mm, F.Cu at (117.8, 125.4)
- added REF**: Via-0.6mm, Dans_Parts:Via-0.6mm, F.Cu at (97.7, 61.1)
- added REF**: Via-0.6mm, Dans_Parts:Via-0.6mm, F.Cu at (31.7, 100.9)
- added REF**: Via-0.6mm, Dans_Parts:Via-0.6mm, F.Cu at (77.8, 41.0)
- added REF**: Via-0.6mm, Dans_Parts:Via-0.6mm, F.Cu at (76.8, 70.7)
- added REF**: Via-0.6mm, Dans_Parts:Via-0.6mm, F.Cu at (70.3, 75.7)
- added REF**: Via-0.6mm, Dans_Parts:Via-0.6mm, F.Cu at (72.2, 72.9)
- added REF**: Via-0.6mm, Dans_Parts:Via-0.6mm, F.Cu at (66.9, 68.6)
- added REF**: Via-0.6mm, Dans_Parts:Via-0.6mm, F.Cu at (61.5, 64.8)
- added REF**: Via-0.6mm, Dans_Parts:Via-0.6mm, F.Cu at (61.0, 68.8)
- added REF**: Via-0.6mm, Dans_Parts:Via-0.6mm, F.Cu at (43.5, 122.1)
- added REF**: Via-0.6mm, Dans_Parts:Via-0.6mm, F.Cu at (29.9, 94.4)
- added REF**: Via-0.6mm, Dans_Parts:Via-0.6mm, F.Cu at (95.9, 61.2)
- added REF**: Via-0.6mm, Dans_Parts:Via-0.6mm, F.Cu at (25.0, 74.6)
- added REF**: Via-0.6mm, Dans_Parts:Via-0.6mm, F.Cu at (68.7, 39.8)
- added REF**: Via-0.6mm, Dans_Parts:Via-0.6mm, F.Cu at (95.6, 67.8)
- added REF**: Via-0.6mm, Dans_Parts:Via-0.6mm, F.Cu at (74.3, 93.8)
- added REF**: Via-0.6mm, Dans_Parts:Via-0.6mm, F.Cu at (74.7, 97.5)
- added REF**: Via-0.6mm, Dans_Parts:Via-0.6mm, F.Cu at (70.0, 107.1)
- added REF**: Via-0.6mm, Dans_Parts:Via-0.6mm, F.Cu at (56.0, 113.5)
- added REF**: Via-0.6mm, Dans_Parts:Via-0.6mm, F.Cu at (47.1, 107.1)
- added REF**: Via-0.6mm, Dans_Parts:Via-0.6mm, F.Cu at (37.6, 125.6)
- added REF**: Via-0.6mm, Dans_Parts:Via-0.6mm, F.Cu at (25.8, 83.1)
- added REF**: Via-0.6mm, Dans_Parts:Via-0.6mm, F.Cu at (97.1, 21.6)
- added REF**: Via-0.6mm, Dans_Parts:Via-0.6mm, F.Cu at (66.4, 33.3)
- added REF**: Via-0.6mm, Dans_Parts:Via-0.6mm, F.Cu at (49.1, 36.4)
- added REF**: Via-0.6mm, Dans_Parts:Via-0.6mm, F.Cu at (65.4, 73.0)
- added REF**: Via-0.6mm, Dans_Parts:Via-0.6mm, F.Cu at (79.3, 98.5)
- added REF**: Via-0.6mm, Dans_Parts:Via-0.6mm, F.Cu at (62.1, 91.6)
- added REF**: Via-0.6mm, Dans_Parts:Via-0.6mm, F.Cu at (56.3, 106.1)
- added REF**: Via-0.6mm, Dans_Parts:Via-0.6mm, F.Cu at (60.4, 95.2)
- added REF**: Via-0.6mm, Dans_Parts:Via-0.6mm, F.Cu at (51.7, 102.0)
- added REF**: Via-0.6mm, Dans_Parts:Via-0.6mm, F.Cu at (32.8, 122.0)
- added REF**: Via-0.6mm, Dans_Parts:Via-0.6mm, F.Cu at (66.4, 125.5)
- added REF**: Via-0.6mm, Dans_Parts:Via-0.6mm, F.Cu at (101.1, 49.4)
- added REF**: Via-0.6mm, Dans_Parts:Via-0.6mm, F.Cu at (80.7, 24.2)
- added REF**: Via-0.6mm, Dans_Parts:Via-0.6mm, F.Cu at (61.8, 22.1)
- added REF**: Via-0.6mm, Dans_Parts:Via-0.6mm, F.Cu at (55.4, 94.5)
- added REF**: Via-0.6mm, Dans_Parts:Via-0.6mm, F.Cu at (110.6, 43.1)
- added REF**: Via-0.6mm, Dans_Parts:Via-0.6mm, F.Cu at (48.3, 47.3)
- added REF**: Via-0.6mm, Dans_Parts:Via-0.6mm, F.Cu at (109.3, 85.2)
- added REF**: Via-0.6mm, Dans_Parts:Via-0.6mm, F.Cu at (119.3, 32.6)
- added REF**: Via-0.6mm, Dans_Parts:Via-0.6mm, F.Cu at (82.8, 73.5)
- added REF**: Via-0.6mm, Dans_Parts:Via-0.6mm, F.Cu at (92.6, 43.5)
- added REF**: Via-0.6mm, Dans_Parts:Via-0.6mm, F.Cu at (85.2, 111.3)
- added REF**: Via-0.6mm, Dans_Parts:Via-0.6mm, F.Cu at (63.4, 100.1)
- added REF**: Via-0.6mm, Dans_Parts:Via-0.6mm, F.Cu at (102.2, 109.2)
- added REF**: Via-0.6mm, Dans_Parts:Via-0.6mm, F.Cu at (64.7, 87.4)
- added REF**: Via-0.6mm, Dans_Parts:Via-0.6mm, F.Cu at (109.0, 109.5)
- added REF**: Via-0.6mm, Dans_Parts:Via-0.6mm, F.Cu at (92.7, 49.0)
- added REF**: Via-0.6mm, Dans_Parts:Via-0.6mm, F.Cu at (61.9, 84.4)
- added REF**: Via-0.6mm, Dans_Parts:Via-0.6mm, F.Cu at (96.9, 55.7)
- added REF**: Via-0.6mm, Dans_Parts:Via-0.6mm, F.Cu at (107.1, 111.4)
- added REF**: Via-0.6mm, Dans_Parts:Via-0.6mm, F.Cu at (83.7, 67.8)
- added REF**: Via-0.6mm, Dans_Parts:Via-0.6mm, F.Cu at (65.2, 84.2)
- added REF**: Via-0.6mm, Dans_Parts:Via-0.6mm, F.Cu at (63.4, 86.0)
- added REF**: Via-0.6mm, Dans_Parts:Via-0.6mm, F.Cu at (98.5, 109.2)
- added REF**: Via-0.6mm, Dans_Parts:Via-0.6mm, F.Cu at (106.9, 107.4)
- added REF**: Via-0.6mm, Dans_Parts:Via-0.6mm, F.Cu at (97.2, 29.3)
- added REF**: Via-0.6mm, Dans_Parts:Via-0.6mm, F.Cu at (97.5, 43.6)
- added REF**: Via-0.6mm, Dans_Parts:Via-0.6mm, F.Cu at (96.3, 48.8)
- added REF**: Via-0.6mm, Dans_Parts:Via-0.6mm, F.Cu at (106.5, 30.8)
- added REF**: Via-0.6mm, Dans_Parts:Via-0.6mm, F.Cu at (104.5, 113.2)
- added REF**: Via-0.6mm, Dans_Parts:Via-0.6mm, F.Cu at (66.6, 85.5)
- added REF**: Via-0.6mm, Dans_Parts:Via-0.6mm, F.Cu at (103.9, 89.9)
- added REF**: Via-0.6mm, Dans_Parts:Via-0.6mm, F.Cu at (63.7, 82.7)
- added REF**: Via-0.6mm, Dans_Parts:Via-0.6mm, F.Cu at (104.8, 109.1)
- added REF**: Via-0.6mm, Dans_Parts:Via-0.6mm, F.Cu at (96.8, 36.1)
- added REF**: Via-0.6mm, Dans_Parts:Via-0.6mm, F.Cu at (83.8, 21.8)
- added REF**: Via-0.6mm, Dans_Parts:Via-0.6mm, F.Cu at (47.7, 94.5)
- added REF**: Via-0.6mm, Dans_Parts:Via-0.6mm, F.Cu at (95.5, 40.1)
- added REF**: Via-0.6mm, Dans_Parts:Via-0.6mm, F.Cu at (36.6, 102.6)
- added REF**: Via-0.6mm, Dans_Parts:Via-0.6mm, F.Cu at (79.1, 69.9)
- added REF**: Via-0.6mm, Dans_Parts:Via-0.6mm, F.Cu at (80.9, 32.5)
- added REF**: Via-0.6mm, Dans_Parts:Via-0.6mm, F.Cu at (90.8, 92.0)
- added REF**: Via-0.6mm, Dans_Parts:Via-0.6mm, F.Cu at (92.3, 107.6)
- added REF**: Via-0.6mm, Dans_Parts:Via-0.6mm, F.Cu at (90.2, 32.4)
- added REF**: Via-0.6mm, Dans_Parts:Via-0.6mm, F.Cu at (98.6, 113.1)
- added REF**: Via-0.6mm, Dans_Parts:Via-0.6mm, F.Cu at (101.0, 21.7)
- added REF**: Via-0.6mm, Dans_Parts:Via-0.6mm, F.Cu at (57.0, 45.4)
- added REF**: Via-0.6mm, Dans_Parts:Via-0.6mm, F.Cu at (95.9, 38.2)
- added REF**: Via-0.6mm, Dans_Parts:Via-0.6mm, F.Cu at (101.2, 38.7)
- added REF**: Via-0.6mm, Dans_Parts:Via-0.6mm, F.Cu at (112.1, 109.3)
- added REF**: Via-0.6mm, Dans_Parts:Via-0.6mm, F.Cu at (112.0, 86.3)
- added REF**: Via-0.6mm, Dans_Parts:Via-0.6mm, F.Cu at (112.1, 90.9)
- added REF**: Via-0.6mm, Dans_Parts:Via-0.6mm, F.Cu at (112.0, 95.4)
- added REF**: Via-0.6mm, Dans_Parts:Via-0.6mm, F.Cu at (94.6, 81.8)
- added REF**: Via-0.6mm, Dans_Parts:Via-0.6mm, F.Cu at (112.0, 100.0)
- added REF**: Via-0.6mm, Dans_Parts:Via-0.6mm, F.Cu at (114.7, 104.6)
- added REF**: Via-0.6mm, Dans_Parts:Via-0.6mm, F.Cu at (88.1, 23.0)
- added REF**: Via-0.6mm, Dans_Parts:Via-0.6mm, F.Cu at (93.6, 66.0)
- added REF**: Via-0.6mm, Dans_Parts:Via-0.6mm, F.Cu at (67.4, 58.9)
- added REF**: Via-0.6mm, Dans_Parts:Via-0.6mm, F.Cu at (63.0, 54.4)
- added REF**: Via-0.6mm, Dans_Parts:Via-0.6mm, F.Cu at (104.6, 106.4)
- added REF**: Via-0.6mm, Dans_Parts:Via-0.6mm, F.Cu at (102.6, 106.4)
- added REF**: Via-0.6mm, Dans_Parts:Via-0.6mm, F.Cu at (64.0, 74.2)
- added REF**: Via-0.6mm, Dans_Parts:Via-0.6mm, F.Cu at (108.3, 93.9)
- added REF**: Via-0.6mm, Dans_Parts:Via-0.6mm, F.Cu at (89.8, 81.7)
- added REF**: Via-0.6mm, Dans_Parts:Via-0.6mm, F.Cu at (108.1, 98.7)
- added REF**: Via-0.6mm, Dans_Parts:Via-0.6mm, F.Cu at (108.1, 104.2)
- added REF**: Via-0.6mm, Dans_Parts:Via-0.6mm, F.Cu at (92.1, 25.7)
- added REF**: Via-0.6mm, Dans_Parts:Via-0.6mm, F.Cu at (76.9, 67.0)
- added REF**: Via-0.6mm, Dans_Parts:Via-0.6mm, F.Cu at (27.7, 28.9)
- added REF**: Via-0.6mm, Dans_Parts:Via-0.6mm, F.Cu at (27.4, 33.6)
- added REF**: Via-0.6mm, Dans_Parts:Via-0.6mm, F.Cu at (104.6, 104.4)
- added REF**: Via-0.6mm, Dans_Parts:Via-0.6mm, F.Cu at (102.6, 104.4)
- added REF**: Via-0.6mm, Dans_Parts:Via-0.6mm, F.Cu at (72.8, 74.8)
- added REF**: Via-0.6mm, Dans_Parts:Via-0.6mm, F.Cu at (108.7, 89.6)
- added REF**: Via-0.6mm, Dans_Parts:Via-0.6mm, F.Cu at (97.6, 65.3)
- added REF**: Via-0.6mm, Dans_Parts:Via-0.6mm, F.Cu at (76.2, 101.9)
- added REF**: Via-0.6mm, Dans_Parts:Via-0.6mm, F.Cu at (83.3, 100.4)
- added REF**: Via-0.6mm, Dans_Parts:Via-0.6mm, F.Cu at (56.8, 42.6)
- added REF**: Via-0.6mm, Dans_Parts:Via-0.6mm, F.Cu at (27.7, 24.1)
- added REF**: Via-0.6mm, Dans_Parts:Via-0.6mm, F.Cu at (25.4, 26.8)
- added REF**: Via-0.6mm, Dans_Parts:Via-0.6mm, F.Cu at (25.4, 30.1)
- added REF**: Via-0.6mm, Dans_Parts:Via-0.6mm, F.Cu at (119.0, 46.6)
- added REF**: Via-0.6mm, Dans_Parts:Via-0.6mm, F.Cu at (107.2, 52.1)
- added REF**: Via-0.6mm, Dans_Parts:Via-0.6mm, F.Cu at (23.4, 112.3)
- added REF**: Via-0.6mm, Dans_Parts:Via-0.6mm, F.Cu at (71.3, 122.7)
- added REF**: Via-0.6mm, Dans_Parts:Via-0.6mm, F.Cu at (96.0, 65.3)
- added REF**: Via-0.6mm, Dans_Parts:Via-0.6mm, F.Cu at (86.2, 122.9)
- added REF**: Via-0.6mm, Dans_Parts:Via-0.6mm, F.Cu at (96.1, 125.7)
- added REF**: Via-0.6mm, Dans_Parts:Via-0.6mm, F.Cu at (115.4, 72.8)
- added REF**: Via-0.6mm, Dans_Parts:Via-0.6mm, F.Cu at (106.2, 73.9)
- added REF**: Via-0.6mm, Dans_Parts:Via-0.6mm, F.Cu at (118.7, 70.4)
- added REF**: Via-0.6mm, Dans_Parts:Via-0.6mm, F.Cu at (119.6, 67.0)
- added REF**: Via-0.6mm, Dans_Parts:Via-0.6mm, F.Cu at (117.4, 60.0)
- added REF**: Via-0.6mm, Dans_Parts:Via-0.6mm, F.Cu at (116.6, 55.2)
- added REF**: Via-0.6mm, Dans_Parts:Via-0.6mm, F.Cu at (23.8, 125.5)
- added REF**: Via-0.6mm, Dans_Parts:Via-0.6mm, F.Cu at (80.3, 125.7)
- R9: value 10 -> 10m
- moved U10 70.6 mm to (39.6, 33.0), turned to 270 degrees
- moved D24 46.5 mm to (36.8, 106.4)
- moved D26 37.9 mm to (115.7, 39.9), turned to 180 degrees
- moved U12 27.5 mm to (100.7, 83.1)
- moved MH2 13.2 mm to (57.8, 137.5)
- moved C3 11.2 mm to (76.7, 58.6), turned to 90 degrees
- moved R3 11.1 mm to (74.0, 58.5), turned to 90 degrees
- moved D21 10.5 mm to (44.3, 114.3)
- moved D28 9.93 mm to (107.0, 68.7)
- moved R5 8.19 mm to (68.8, 62.1), turned to 0 degrees
- moved R8 7.43 mm to (68.8, 54.9), turned to 0 degrees
- moved U11 7.40 mm to (100.7, 76.0), turned to 0 degrees
- moved D34 6.78 mm to (61.0, 61.1), turned to 90 degrees
- moved D20 6.63 mm to (50.4, 112.0)
- moved D19 5.88 mm to (61.5, 112.7)
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Connections:
- D21 pad 1: UART_3_TX -> RESET_PI_3
- D21 pad 3: RESET_PI_3 -> UART_3_TX
- D28 pad 4: IMU_MISO -> IMU_MOSI
- D28 pad 6: IMU_MOSI -> IMU_MISO
- D29 pad 3: PWM_CURRENT_CTRL -> MOTOR_DIRECTION_5
- D29 pad 4: MOTOR_DIRECTION_5 -> PWM_CURRENT_CTRL
- J7 pad 1: MEAS_SPEED -> MEAS_CURRENT
- J7 pad 2: MEAS_CURRENT -> MEAS_SPEED
- U10 pad 3: MCELL3 -> MCELL2
- U10 pad 7: CELL1 -> Net-(U10-Pad7)
- U10 pad 9: MCELL2 -> MCELL3
- U11 pad 1: CELL2 -> CELL4
- U11 pad 3: CELL4 -> CELL3
- U11 pad 7: CELL5 -> CELL2
- U11 pad 9: CELL3 -> CELL1
- U12 pad 1: CELL6 -> MEAS_SPEED
- U12 pad 3: MEAS_SPEED -> CELL6
- U12 pad 7: Net-(U12-Pad7) -> CELL5
- U5 pad 30: CELL1 -> CELL6
- U5 pad 31: CELL2 -> CELL5
- U5 pad 32: CELL3 -> CELL4
- U5 pad 33: CELL4 -> CELL3
- U5 pad 34: CELL5 -> CELL2
- U5 pad 35: CELL6 -> CELL1
Routing:
- net +3.3V: track 0.00 -> 171.4 mm, vias 0 -> 5
- net TEENSY_SDA: track 0.00 -> 158.2 mm, vias 0 -> 3
- net MCELL1: track 0.00 -> 153.3 mm, vias 0 -> 1
- net TEENSY_SCL: track 0.00 -> 153.1 mm, vias 0 -> 2
- net MCELL2: track 0.00 -> 151.2 mm, vias 0 -> 1
- net MCELL3: track 0.00 -> 144.6 mm, vias 0 -> 1
- net GND: track 0.00 -> 126.5 mm, vias 0 -> 22
- net RESET_PI_4: track 0.00 -> 121.3 mm, vias 0 -> 2
- net IMU_SCLK: track 0.00 -> 119.8 mm, vias 0 -> 2
- net UART_4_RX: track 0.00 -> 113.0 mm, vias 0 -> 2
- net UART_4_TX: track 0.00 -> 112.1 mm, vias 0 -> 2
- net +6.5V: track 0.00 -> 111.9 mm, vias 0 -> 1
- net 2S_Backup_IN: track 0.00 -> 96.4 mm, vias 0 -> 1
- net MSP_GPIO_0: track 0.00 -> 94.4 mm, vias 0 -> 1
- net MULTIPLEX_A1: track 0.00 -> 89.1 mm, vias 0 -> 1
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- added copper zone on 3V3, net +3.3V
- added copper zone on B.Cu, net +5V
- added copper zone on F.Cu, net GND
- added copper zone on GND, net GND
Other:
- copper layers 2 -> 4
- net class 2A added: clearance 0.2, trace_width 1, via_dia 1.2, via_drill 1.1
- net class Small Clearance added: clearance 0.1, trace_width 0.2, via_dia 0.4, via_drill 0.3
- net class ~4A added: clearance 0.3, trace_width 1.5, via_dia 4, via_drill 2
- rule trace_min: 0.2 -> 0.15

Commit message: Board Completed. Needs Review
Parts:
- removed J20: RESET_VIDEO_PI, Dans_Parts:2-Pin_Molex_Horizontal
- removed the REF** at (94.5, 79.6)
- removed the REF** at (89.8, 79.7)
- removed the REF** at (64.7, 87.4)
- removed the REF** at (61.9, 84.4)
- removed the REF** at (65.2, 84.2)
- removed the REF** at (63.4, 86.0)
- removed the REF** at (97.5, 43.6)
- removed the REF** at (66.6, 85.5)
- removed the REF** at (63.7, 82.7)
- removed the REF** at (94.6, 81.8)
- removed the REF** at (89.8, 81.7)
- added W1: TEST_1P, Connect:PINTST, F.Cu at (57.9, 114.3)
- added W12: TEST_1P, Connect:PINTST, F.Cu at (58.0, 110.8)
- added W13: TEST_1P, Connect:PINTST, F.Cu at (29.9, 110.5)
- added W14: TEST_1P, Connect:PINTST, F.Cu at (93.1, 109.5)
- added W17: TEST_1P, Connect:PINTST, F.Cu at (36.8, 45.6)
- added W18: TEST_1P, Connect:PINTST, F.Cu at (42.9, 94.7)
- added W2: TEST_1P, Connect:PINTST, F.Cu at (26.2, 110.7)
- added W21: TEST_1P, Connect:PINTST, F.Cu at (57.1, 103.7)
- added W23: TEST_1P, Connect:PINTST, F.Cu at (46.1, 107.0)
- added W24: TEST_1P, Connect:PINTST, F.Cu at (68.9, 121.9)
- added W27: TEST_1P, Connect:PINTST, F.Cu at (106.5, 48.7)
- added W28: TEST_1P, Connect:PINTST, F.Cu at (81.6, 71.5)
- added W29: TEST_1P, Connect:PINTST, F.Cu at (36.0, 101.9)
- added W3: TEST_1P, Connect:PINTST, F.Cu at (83.8, 116.1)
- added W32: TEST_1P, Connect:PINTST, F.Cu at (52.4, 103.6)
- added W34: TEST_1P, Connect:PINTST, F.Cu at (50.3, 107.0)
- added W35: TEST_1P, Connect:PINTST, F.Cu at (54.6, 107.1)
- added W38: TEST_1P, Connect:PINTST, F.Cu at (107.1, 59.3)
- added W39: TEST_1P, Connect:PINTST, F.Cu at (49.1, 37.7)
- added W43: TEST_1P, Connect:PINTST, F.Cu at (41.0, 104.3)
- added W45: TEST_1P, Connect:PINTST, F.Cu at (45.1, 118.3)
- added W46: TEST_1P, Connect:PINTST, F.Cu at (86.0, 114.4)
- added W49: TEST_1P, Connect:PINTST, F.Cu at (105.7, 71.9)
- added W50: TEST_1P, Connect:PINTST, F.Cu at (66.1, 57.0)
- added W54: TEST_1P, Connect:PINTST, F.Cu at (39.3, 105.9)
- added W55: TEST_1P, Connect:PINTST, F.Cu at (27.2, 94.5)
- added W56: TEST_1P, Connect:PINTST, F.Cu at (45.1, 123.5)
- added W57: TEST_1P, Connect:PINTST, F.Cu at (59.4, 107.3)
- added W6: TEST_1P, Connect:PINTST, F.Cu at (28.9, 36.3)
- added W60: TEST_1P, Connect:PINTST, F.Cu at (105.7, 74.1)
- added W61: TEST_1P, Connect:PINTST, F.Cu at (60.9, 83.7)
- added W65: TEST_1P, Connect:PINTST, F.Cu at (116.8, 42.8)
- added W7: TEST_1P, Connect:PINTST, F.Cu at (62.5, 85.4)
- R38: value 10kR -> 10k
- moved MH2 127.6 mm to (117.6, 24.8)
- moved J11 90.0 mm to (113.7, 122.7), turned to 0 degrees
- moved D24 70.6 mm to (106.7, 115.7)
- moved REF** 23.8 mm to (96.1, 115.8)
- moved REF** 13.3 mm to (40.4, 86.1)
- moved REF** 10.7 mm to (100.1, 113.4)
- moved REF** 9.82 mm to (27.6, 98.7)
- moved REF** 5.36 mm to (60.0, 102.2)
- moved REF** 4.33 mm to (109.9, 71.7)
- moved REF** 3.51 mm to (22.3, 98.6)
- moved REF** 3.15 mm to (96.7, 66.5)
- moved REF** 2.61 mm to (54.1, 101.0)
- moved REF** 1.80 mm to (47.5, 35.6)
- moved REF** 1.75 mm to (43.7, 101.2)
- moved R14 1.69 mm to (41.6, 100.6)
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Connections:
- U8 pad 67: RESET_VIDEO_PI -> Net-(U8-Pad67)
Routing:
- net RESET_VIDEO_PI: track 52.8 -> 0.00 mm, vias 2 -> 0
- net UART_4_RX: track 113.0 -> 64.7 mm
- net UART_4_TX: track 112.1 -> 66.6 mm
- net RESET_PI_4: track 121.3 -> 77.7 mm
- net COMMS_MISO: track 40.7 -> 69.6 mm, vias 2 -> 3
- net TEENSY_SCL: track 153.1 -> 174.3 mm
- net TEENSY_SDA: track 158.2 -> 176.5 mm
- net MULTIPLEX_A0: track 87.4 -> 102.2 mm
- net COMMS_MOSI: track 39.9 -> 54.3 mm
- net UART_2_TX: track 44.6 -> 58.3 mm
- net COMMS_SCLK: track 44.6 -> 57.9 mm
- net COMMS_CS: track 57.7 -> 70.8 mm
- net RESET_PI_3: track 61.1 -> 71.0 mm
- net UART_3_RX: track 63.4 -> 73.1 mm
- net MULTIPLEX_A1: track 89.1 -> 98.7 mm
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Other:
- board text added: "*Made on Earth by humans*"
- board text added: "Designer: Daniel Mitchell"
- board text added: "HABIP 2018"
- board text added: "RIT Senior Design"
- board text removed: "Slide Switch: 3S (Above) 2S (Below)"

Commit message: Added BOM, Couple Fixes, Couple Misc Documents
Parts:
- removed the REF** at (110.6, 43.1)
- removed the REF** at (92.3, 107.6)
- removed U9: ASEMB-24MHZ-XY-T, Dans_Parts:ASEMB-24MHZ
- removed W49: TEST_1P, Connect:PINTST
- added REF**: Via-0.6mm, Dans_Parts:Via-0.6mm, F.Cu at (94.4, 66.2)
- added Y2: ASEMB-24MHZ-XY-T, Dans_Parts:ASEMB-24MHZ, F.Cu at (82.8, 86.1)
- C18: value 10uF -> 0.1uF
- C20, C23, C27, C28, C29: value 100nF -> 0.1uF
- C24, C33: value 1000pF -> 1nF
- D11: value SBRT5A50SA-13 -> CDBA540-HF
- R37: value 10kR -> 10k
- R39, R55: value 80 -> 100
Connections:
- D27 pad 4: MULTIPLEX_A1 -> Net-(D27-Pad4)
- D27 pad 6: MULTIPLEX_A0 -> Net-(D27-Pad6)
- J5 pad 2: MULTIPLEX_A1 -> MSP_GPIO_CB
- J5 pad 3: MULTIPLEX_A0 -> +3.3V
- R40 pad 1: +5V -> +3.3V
- R46 pad 1: +5V -> +3.3V
- U8 pad 17: MULTIPLEX_A0 -> Net-(U8-Pad17)
- U8 pad 18: MULTIPLEX_A1 -> MSP_GPIO_CB
- W60 pad 1: MULTIPLEX_A1 -> MSP_GPIO_CB
Routing:
- net MULTIPLEX_A0: track 102.2 -> 0.00 mm, vias 2 -> 0
- net MULTIPLEX_A1: track 98.7 -> 0.00 mm, vias 1 -> 0
- net MSP_GPIO_CB: track 0.00 -> 90.5 mm, vias 0 -> 1
- net +3.3V: track 170.3 -> 187.0 mm, vias 5 -> 7
- net +5V: track 71.4 -> 66.2 mm
- net IMU_SCLK: track 119.8 -> 122.3 mm
- net GND: track 127.3 -> 129.1 mm
