File: PCB/MainBoardV2/mainBoardV2.sch (KiCad schematic (older format))
At the start: 27 parts, among them J1 Pi0_1, J10 Backup_Battery, J11 External_Temp, J12 Comms_I2C, J13 Main_Monitoring, J14 2S_Primary_Batt, J15 2S_Backup_Batt, J16 Programming, J17 To_Balloon, J18 Motor_Batt_Monitoring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

Commit message: Layout Done - Needs TPs Still
Parts:
- added J21: Ethernet_Switch_PWR, Dans_Parts:2-Pin_Molex_Horizontal, symbol CONN_01X02
Connections:
- net GND: now also J21.1 (P1)
- net MEAS_CURRENT: now also J7.1 (P1); no longer J7.2 (P2)
- net MEAS_SPEED: now also J7.2 (P2); no longer J7.1 (P1)
- new net +5V: J21.2 (P2)
Other:
- note added: "Mounting\nHoles &\nSwitch PWR"
- note added: "Pi3 Reset"
- note removed: "Mounting\nHoles"
- note removed: "Video Pi Reset"
- moved on the sheet: J12, J20, J9, MH1, MH2, MH3, MH4

Commit message: Board Completed. Needs Review
Parts:
- removed J20: RESET_VIDEO_PI, Dans_Parts:2-Pin_Molex_Horizontal, symbol CONN_01X02
Other:
- note added: "Mounting\nHoles"
- note added: "Switch PWR"
- note removed: "Mounting\nHoles &\nSwitch PWR"
- note removed: "Pi3 Reset"
- moved on the sheet: J12, J9, MH1, MH2, MH3, MH4
Changed lines of the file:
@@
 L CONN_01X05 J9
 U 1 1 5A011DB4
-P 5400 5950
-F 0 "J9" H 5400 6250 50  0000 C CNN
-F 1 "Comms_SPI" V 5500 5950 50  0000 C CNN
-F 2 "Dans_Parts:6-Pin_Molex_Horizontal" H 5400 5950 50  0001 C CNN
-F 3 "" H 5400 5950 50  0000 C CNN
-	1    5400 5950
+P 3550 5950
+F 0 "J9" H 3550 6250 50  0000 C CNN
+F 1 "Comms_SPI" V 3650 5950 50  0000 C CNN
+F 2 "Dans_Parts:6-Pin_Molex_Horizontal" H 3550 5950 50  0001 C CNN
+F 3 "" H 3550 5950 50  0000 C CNN
+	1    3550 5950
 	-1   0    0    -1
 $EndComp
@@
 L GND #PWR05
 U 1 1 5A011EEC
-P 5650 6200
-F 0 "#PWR05" H 5650 5950 50  0001 C CNN
-F 1 "GND" H 5650 6050 50  0000 C CNN
-F 2 "" H 5650 6200 50  0000 C CNN
-F 3 "" H 5650 6200 50  0000 C CNN
-	1    5650 6200
-	1    0    0    -1
-$EndComp
-Text GLabel 5600 5750 2    39   Input ~ 0
+P 3800 6200
+F 0 "#PWR05" H 3800 5950 50  0001 C CNN
+F 1 "GND" H 3800 6050 50  0000 C CNN
+F 2 "" H 3800 6200 50  0000 C CNN
+F 3 "" H 3800 6200 50  0000 C CNN
+	1    3800 6200
+	1    0    0    -1
+$EndComp
+Text GLabel 3750 5750 2    39   Input ~ 0
 COMMS_CS
-Text GLabel 5600 5850 2    39   Input ~ 0
+Text GLabel 3750 5850 2    39   Input ~ 0
 COMMS_SCLK
-Text GLabel 5600 5950 2    39   Input ~ 0
+Text GLabel 3750 5950 2    39   Input ~ 0
 COMMS_MISO
-Text GLabel 5600 6050 2    39   Input ~ 0
+Text GLabel 3750 6050 2    39   Input ~ 0
 COMMS_MOSI
-Text Notes 5150 5500 0    197  ~ 0
+Text Notes 3300 5500 0    197  ~ 0
 Comms Board
 $Comp
 L GND #PWR06
 U 1 1 5A01B32C
-P 6750 6150
-F 0 "#PWR06" H 6750 5900 50  0001 C CNN
-F 1 "GND" H 6750 6000 50  0000 C CNN
-F 2 "" H 6750 6150 50  0000 C CNN
-F 3 "" H 6750 6150 50  0000 C CNN
-	1    6750 6150
-	1    0    0    -1
-$EndComp
-Text GLabel 6700 5900 2    39   Input ~ 0
+P 4900 6150
+F 0 "#PWR06" H 4900 5900 50  0001 C CNN
+F 1 "GND" H 4900 6000 50  0000 C CNN
+F 2 "" H 4900 6150 50  0000 C CNN
+F 3 "" H 4900 6150 50  0000 C CNN
+	1    4900 6150
+	1    0    0    -1
+$EndComp
+Text GLabel 4850 5900 2    39   Input ~ 0
 HOST_SCL
-Text GLabel 6700 6000 2    39   Input ~ 0
+Text GLabel 4850 6000 2    39   Input ~ 0
 HOST_SDA
 Text Notes 5050 4250 0    197  ~ 0
@@
 L CONN_01X04 J12
 U 1 1 5A01DD06
-P 6500 5950
-F 0 "J12" H 6500 6200 50  0000 C CNN
-F 1 "Comms_I2C" V 6600 5950 50  0000 C CNN
-F 2 "Dans_Parts:4-Pin_Molex_Horizontal" H 6500 5950 50  0001 C CNN
-F 3 "" H 6500 5950 50  0000 C CNN
-	1    6500 5950
+P 4650 5950
+F 0 "J12" H 4650 6200 50  0000 C CNN
+F 1 "Comms_I2C" V 4750 5950 50  0000 C CNN
+F 2 "Dans_Parts:4-Pin_Molex_Horizontal" H 4650 5950 50  0001 C CNN
+F 3 "" H 4650 5950 50  0000 C CNN
+	1    4650 5950
 	-1   0    0    -1
 $EndComp
@@
 Text GLabel 7900 2800 2    39   Input ~ 0
 +3.3V
-Text GLabel 6700 5800 2    39   Input ~ 0
+Text GLabel 4850 5800 2    39   Input ~ 0
 +3.3V
 $Sheet
@@
 F1 "MSP430.sch" 79
 $EndSheet
-$Comp
-L CONN_01X02 J20
-U 1 1 5A73A347
-P 3900 5800
-F 0 "J20" H 3900 5650 50  0000 C CNN
-F 1 "RESET_VIDEO_PI" V 4000 5800 50  0000 C CNN
-F 2 "Dans_Parts:2-Pin_Molex_Horizontal" H 3900 5800 50  0001 C CNN
-F 3 "" H 3900 5800 50  0000 C CNN
-	1    3900 5800
-	-1   0    0    1
-$EndComp
-$Comp
-L GND #PWR020
-U 1 1 5A73A4F9
-P 4150 5900
-F 0 "#PWR020" H 4150 5650 50  0001 C CNN
-F 1 "GND" H 4150 5750 50  0000 C CNN
-F 2 "" H 4150 5900 50  0000 C CNN
-F 3 "" H 4150 5900 50  0000 C CNN
-	1    4150 5900
-	1    0    0    -1
-$EndComp
-Wire Wire Line
-	4150 5850 4100 5850
-Wire Wire Line
-	4150 5900 4150 5850
 Wire Wire Line
 	8750 3350 8700 3350
@@
 	5000 3950 7050 3950
 Wire Notes Line
-	5100 6450 5100 5200
-Wire Notes Line
-	7250 6450 5100 6450
-Wire Notes Line
-	7250 5200 7250 6450
-Wire Notes Line
-	5100 5200 7250 5200
-Wire Wire Line
-	6750 6100 6700 6100
-Wire Wire Line
-	6750 6150 6750 6100
-Wire Wire Line
-	5650 6150 5600 6150
-Wire Wire Line
-	5650 6200 5650 6150
+	3250 6450 3250 5200
+Wire Notes Line
+	5400 6450 3250 6450
+Wire Notes Line
+	5400 5200 5400 6450
+Wire Notes Line
+	3250 5200 5400 5200
+Wire Wire Line
+	4900 6100 4850 6100
+Wire Wire Line
+	4900 6150 4900 6100
+Wire Wire Line
+	3800 6150 3750 6150
+Wire Wire Line
+	3800 6200 3800 6150
 Wire Notes Line
 	7500 5000 7500 3900
@@
 Wire Notes Line
 	3150 500  3150 7800
-Text GLabel 4100 5750 2    39   Input ~ 0
-RESET_VIDEO_PI
 Text Notes 5450 1050 0    197  ~ 0
 3-Cell Batts
@@
 Wire Notes Line
 	9400 1900 9400 650
-Text Notes 3450 5450 0    197  ~ 0
-Pi3 Reset
-Wire Notes Line
-	3400 5200 4950 5200
-Wire Notes Line
-	4950 5200 4950 6150
-Wire Notes Line
-	4950 6150 3400 6150
-Wire Notes Line
-	3400 6150 3400 5200
 Wire Wire Line
 	6100 6850 6100 6950
@@
 L Mounting_Hole_Eighth_Inch MH1
 U 1 1 5A777134
-P 9550 5500
-F 0 "MH1" H 9556 5649 39  0000 C CNN
-F 1 "GND" H 9650 5400 39  0000 C CNN
-F 2 "Dans_Parts:Mounting_Hole_Eighth_Inch" H 9550 5500 39  0001 C CNN
-F 3 "" H 9550 5500 39  0001 C CNN
-	1    9550 5500
-	1    0    0    -1
-$EndComp
-$Comp
-L GND #PWR021
+P 7400 5500
+F 0 "MH1" H 7406 5649 39  0000 C CNN
+F 1 "GND" H 7500 5400 39  0000 C CNN
+F 2 "Dans_Parts:Mounting_Hole_Eighth_Inch" H 7400 5500 39  0001 C CNN
+F 3 "" H 7400 5500 39  0001 C CNN
+	1    7400 5500
+	1    0    0    -1
+$EndComp
+$Comp
+L GND #PWR020
 U 1 1 5A777D3D
-P 9550 5650
-F 0 "#PWR021" H 9550 5400 50  0001 C CNN
-F 1 "GND" H 9550 5500 50  0000 C CNN
-F 2 "" H 9550 5650 50  0000 C CNN
-F 3 "" H 9550 5650 50  0000 C CNN
-	1    9550 5650
+P 7400 5650
+F 0 "#PWR020" H 7400 5400 50  0001 C CNN
+F 1 "GND" H 7400 5500 50  0000 C CNN
+F 2 "" H 7400 5650 50  0000 C CNN
+F 3 "" H 7400 5650 50  0000 C CNN
+	1    7400 5650
 	1    0    0    -1
 $EndComp
@@
 L Mounting_Hole_Eighth_Inch MH3
 U 1 1 5A777F0E
-P 10000 5500
-F 0 "MH3" H 10006 5649 39  0000 C CNN
-F 1 "GND" H 10100 5400 39  0000 C CNN
-F 2 "Dans_Parts:Mounting_Hole_Eighth_Inch" H 10000 5500 39  0001 C CNN
-F 3 "" H 10000 5500 39  0001 C CNN
-	1    10000 5500
-	1    0    0    -1
-$EndComp
-$Comp
-L GND #PWR022
+P 7850 5500
+F 0 "MH3" H 7856 5649 39  0000 C CNN
+F 1 "GND" H 7950 5400 39  0000 C CNN
+F 2 "Dans_Parts:Mounting_Hole_Eighth_Inch" H 7850 5500 39  0001 C CNN
+F 3 "" H 7850 5500 39  0001 C CNN
+	1    7850 5500
+	1    0    0    -1
+$EndComp
+$Comp
+L GND #PWR021
 U 1 1 5A777F14
-P 10000 5650
-F 0 "#PWR022" H 10000 5400 50  0001 C CNN
-F 1 "GND" H 10000 5500 50  0000 C CNN
-F 2 "" H 10000 5650 50  0000 C CNN
-F 3 "" H 10000 5650 50  0000 C CNN
-	1    10000 5650
+P 7850 5650
+F 0 "#PWR021" H 7850 5400 50  0001 C CNN
+F 1 "GND" H 7850 5500 50  0000 C CNN
+F 2 "" H 7850 5650 50  0000 C CNN
+F 3 "" H 7850 5650 50  0000 C CNN
+	1    7850 5650
 	1    0    0    -1
 $EndComp
@@
 L Mounting_Hole_Eighth_Inch MH2
 U 1 1 5A77802D
-P 9550 6050
-F 0 "MH2" H 9556 6199 39  0000 C CNN
-F 1 "GND" H 9650 5950 39  0000 C CNN
-F 2 "Dans_Parts:Mounting_Hole_Eighth_Inch" H 9550 6050 39  0001 C CNN
-F 3 "" H 9550 6050 39  0001 C CNN
-	1    9550 6050
-	1    0    0    -1
-$EndComp
-$Comp
-L GND #PWR023
+P 7400 6050
+F 0 "MH2" H 7406 6199 39  0000 C CNN
+F 1 "GND" H 7500 5950 39  0000 C CNN
+F 2 "Dans_Parts:Mounting_Hole_Eighth_Inch" H 7400 6050 39  0001 C CNN
+F 3 "" H 7400 6050 39  0001 C CNN
+	1    7400 6050
+	1    0    0    -1
+$EndComp
+$Comp
+L GND #PWR022
 U 1 1 5A778033
-P 9550 6200
-F 0 "#PWR023" H 9550 5950 50  0001 C CNN
-F 1 "GND" H 9550 6050 50  0000 C CNN
-F 2 "" H 9550 6200 50  0000 C CNN
-F 3 "" H 9550 6200 50  0000 C CNN
-	1    9550 6200
+P 7400 6200
+F 0 "#PWR022" H 7400 5950 50  0001 C CNN
+F 1 "GND" H 7400 6050 50  0000 C CNN
+F 2 "" H 7400 6200 50  0000 C CNN
+F 3 "" H 7400 6200 50  0000 C CNN
+	1    7400 6200
 	1    0    0    -1
 $EndComp
@@
 L Mounting_Hole_Eighth_Inch MH4
 U 1 1 5A778039
-P 10000 6050
-F 0 "MH4" H 10006 6199 39  0000 C CNN
-F 1 "GND" H 10100 5950 39  0000 C CNN
-F 2 "Dans_Parts:Mounting_Hole_Eighth_Inch" H 10000 6050 39  0001 C CNN
-F 3 "" H 10000 6050 39  0001 C CNN
-	1    10000 6050
-	1    0    0    -1
-$EndComp
-$Comp
-L GND #PWR024
+P 7850 6050
+F 0 "MH4" H 7856 6199 39  0000 C CNN
+F 1 "GND" H 7950 5950 39  0000 C CNN
+F 2 "Dans_Parts:Mounting_Hole_Eighth_Inch" H 7850 6050 39  0001 C CNN
+F 3 "" H 7850 6050 39  0001 C CNN
+	1    7850 6050
+	1    0    0    -1
+$EndComp
+$Comp
+L GND #PWR023
 U 1 1 5A77803F
-P 10000 6200
-F 0 "#PWR024" H 10000 5950 50  0001 C CNN
-F 1 "GND" H 10000 6050 50  0000 C CNN
-F 2 "" H 10000 6200 50  0000 C CNN
-F 3 "" H 10000 6200 50  0000 C CNN
-	1    10000 6200
-	1    0    0    -1
-$EndComp
-Text Notes 7500 6300 0    197  ~ 39
-Mounting\nHoles &\nSwitch PWR
-Wire Notes Line
-	7400 6550 7400 5200
-Wire Notes Line
-	7400 5200 11200 5200
+P 7850 6200
+F 0 "#PWR023" H 7850 5950 50  0001 C CNN
+F 1 "GND" H 7850 6050 50  0000 C CNN
+F 2 "" H 7850 6200 50  0000 C CNN
+F 3 "" H 7850 6200 50  0000 C CNN
+	1    7850 6200
+	1    0    0    -1
+$EndComp
+Text Notes 5800 6250 0    197  ~ 39
+Mounting\nHoles
+Wire Notes Line
+	5600 6550 5600 5200
+Wire Notes Line
+	5600 5200 11200 5200
 $Comp
 L CONN_01X02 J19
@@
 $EndComp
 $Comp
-L GND #PWR025
+L GND #PWR024
 U 1 1 5A7B9767
 P 10750 5950
-F 0 "#PWR025" H 10750 5700 50  0001 C CNN
+F 0 "#PWR024" H 10750 5700 50  0001 C CNN
 F 1 "GND" H 10750 5800 50  0000 C CNN
 F 2 "" H 10750 5950 50  0000 C CNN
@@
 Text GLabel 10700 5800 2    39   Input ~ 0
 +5V
+Text Notes 8400 5950 0    197  ~ 39
+Switch PWR
+Wire Notes Line
+	8200 5200 8200 6550
 $EndSCHEMATC

Commit message: Updated a couple nets to the proper voltage and re-plotted the schematic
Other:
- note added: "Network\nSwitch PWR"
- note removed: "Switch PWR"
Changed lines of the file:
@@
 Text GLabel 10700 5800 2    39   Input ~ 0
 +5V
-Text Notes 8400 5950 0    197  ~ 39
-Switch PWR
+Text Notes 8400 6150 0    197  ~ 39
+Network\nSwitch PWR
 Wire Notes Line
 	8200 5200 8200 6550

Commit message: Added BOM, Couple Fixes, Couple Misc Documents
Connections:
- net MULTIPLEX_A0 is gone; now on net +3.3V: J5.3 (P3)
- net MULTIPLEX_A1 renamed MSP_GPIO_CB
Changed lines of the file:
@@
 	-1   0    0    1
 $EndComp
-Text GLabel 8700 3150 2    39   Input ~ 0
-MULTIPLEX_A0
-Text GLabel 8700 3250 2    39   Input ~ 0
-MULTIPLEX_A1
 Text GLabel 7900 2800 2    39   Input ~ 0
 +3.3V
@@
 Wire Notes Line
 	8200 5200 8200 6550
+Text GLabel 8700 3150 2    39   Input ~ 0
++3.3V
+Text GLabel 8700 3250 2    39   Input ~ 0
+MSP_GPIO_CB
 $EndSCHEMATC
